Commit message: nwm co zrobilem wiecej od cb

File: lab2/urdf/bogson_template.urdf.xacro (robot description, xacro)
@@ -1,6 +1,16 @@
+<?xml version="1.0" ?>
 <robot name="bogson" xmlns:xacro="http://www.ros.org/wiki/xacro">
-    <xacro:property name="DH" value="${load_yaml('DH.yaml')}"/>
-    <xacro:property name="params" value="${load_yaml('rpy.yaml')}"/>
-    <xacro:macro name="link" params="name originxyz dimensions">
+<!--     <xacro:property name="DH" value="${load_yaml('DH.yaml')}"/>
+    <xacro:property name="params" value="${load_yaml('rpy.yaml')}"/> -->
+    <xacro:macro name="joint" params=" name type axis parent child originxyz originrpy">
+        <joint name="${name}" type="${type}">
+            <axis xyz="${axis}"/>
+            <limit upper="3.1415" lower="-3.1415" effort="10" velocity="2" />
+            <parent link="${parent}"/>
+            <child link="${child}"/>
+            <origin xyz="${originxyz}" rpy="${originrpy}"/>
+        </joint>
+    </xacro:macro>
+    <xacro:macro name="m_link" params=" name originxyz dimensions">
         <link name="${name}">
             <visual>
@@ -15,12 +25,3 @@
         </link>
     </xacro:macro>
-    <xacro:macro name="joint" params=" name type axis parent child originxyz originrpy">
-        <joint name="${name}" type="${type}">
-            <axis xyz="${axis}"/>
-            <limit upper="3.1415" lower="-3.1415" effort="10" velocity="2" />
-            <parent link="${parent}"/>
-            <child link="${child}"/>
-            <origin xyz="${originxyz}" rpy="${originrpy}"/>
-        </joint>
-    </xacro:macro>
 </robot>
