Commit message: Revert "nwm co zrobilem wiecej od cb"
This reverts commit 638eae5937e299c76e8508bce1f254a2f20f29ab.

File: lab2/urdf/bogson.urdf.xacro (robot description, xacro)
@@ -1,17 +1,19 @@
-<?xml version="1.0" ?>
 <robot name="bogson" xmlns:xacro="http://www.ros.org/wiki/xacro">
   <!-- BGN - Include -->
   <xacro:include filename="$(find lab2)/bogson_template.urdf.xacro" />
-  <xacro:include filename="$(find lab2)/parameters.urdf.xacro" />
   <!-- END - Include -->
+  <xacro:property name="parameters" value="${load_yaml(find lab2)/parameters.yaml)}" />
+  <xacro:property name="a1" value="${parameters['a1']}" />
+  <xacro:property name="a2" value="${parameters['a2']}" />
+  <xacro:property name="a3" value="${parameters['a3']}" />
   <!-- BGN - Robot description -->
-  <xacro:m_link name="base"
+  <xacro:link name="base"
     originxyz="0 0 0"
     dimensions="5 5 1">
-  </xacro:m_link>
-  <xacro:m_link name="link1"
-    originxyz="0 0 ${ajeden/2}"
-    dimensions="1 1 ${ajeden}">
-  </xacro:m_link>
+  </xacro:link>
+  <xacro:link name="link1"
+    originxyz="0 0 ${a1/2}"
+    dimensions="1 1 ${a1}">
+  </xacro:link>
   <xacro:joint name="base_to_link1"
     type="revolute"
@@ -22,37 +24,37 @@
     child="link1">
   </xacro:joint>
-  <xacro:m_link name="link2"
-    originxyz="0 0 ${adwa/2}"
-    dimensions="1 1 ${adwa}">
-  </xacro:m_link>
+  <xacro:link name="link2"
+    originxyz="0 0 ${a2/2}"
+    dimensions="1 1 ${a2}">
+  </xacro:link>
   <xacro:joint name="link1_to_link2"
     type="revolute"
     axis="0 0 1"
     originrpy="0 0 ${1.57075}"
-    originxyz="0 0 ${ajeden}"
+    originxyz="0 0 ${a1}"
     parent="link1"
     child="link2">
   </xacro:joint>
-  <xacro:m_link name="link3"
-    originxyz="0 0 ${atrzy/2}"
-    dimensions="1 1 ${atrzy}">
-  </xacro:m_link>
+  <xacro:link name="link3"
+    originxyz="0 0 ${a3/2}"
+    dimensions="1 1 ${a3}">
+  </xacro:link>
   <xacro:joint name="link2_to_link3"
     type="revolute"
     axis="0 0 1"
     originrpy="0 0 0"
-    originxyz="0 0 ${adwa}"
+    originxyz="0 0 ${a2}"
     parent="link2"
     child="link3">
   </xacro:joint>
-  <xacro:m_link name="narzedzie"
+  <xacro:link name="narzedzie"
     originxyz="0 0 0.5"
     dimensions = "1 1 1">
-  </xacro:m_link>
+  </xacro:link>
   <xacro:joint name="link3_to_narzedzie"
     type="revolute"
     axis="0 0 1"
     originrpy="0 0 0"
-    originxyz="0 0 ${atrzy}"
+    originxyz="0 0 ${a3}"
     parent="link3"
     child="narzedzie">

File: lab2/urdf/bogson_template.urdf.xacro (robot description, xacro)
@@ -1,16 +1,6 @@
-<?xml version="1.0" ?>
 <robot name="bogson" xmlns:xacro="http://www.ros.org/wiki/xacro">
-<!--     <xacro:property name="DH" value="${load_yaml('DH.yaml')}"/>
-    <xacro:property name="params" value="${load_yaml('rpy.yaml')}"/> -->
-    <xacro:macro name="joint" params=" name type axis parent child originxyz originrpy">
-        <joint name="${name}" type="${type}">
-            <axis xyz="${axis}"/>
-            <limit upper="3.1415" lower="-3.1415" effort="10" velocity="2" />
-            <parent link="${parent}"/>
-            <child link="${child}"/>
-            <origin xyz="${originxyz}" rpy="${originrpy}"/>
-        </joint>
-    </xacro:macro>
-    <xacro:macro name="m_link" params=" name originxyz dimensions">
+    <xacro:property name="DH" value="${load_yaml('DH.yaml')}"/>
+    <xacro:property name="params" value="${load_yaml('rpy.yaml')}"/>
+    <xacro:macro name="link" params="name originxyz dimensions">
         <link name="${name}">
             <visual>
@@ -25,3 +15,12 @@
         </link>
     </xacro:macro>
+    <xacro:macro name="joint" params=" name type axis parent child originxyz originrpy">
+        <joint name="${name}" type="${type}">
+            <axis xyz="${axis}"/>
+            <limit upper="3.1415" lower="-3.1415" effort="10" velocity="2" />
+            <parent link="${parent}"/>
+            <child link="${child}"/>
+            <origin xyz="${originxyz}" rpy="${originrpy}"/>
+        </joint>
+    </xacro:macro>
 </robot>

Commit message: już powinno xacro działąć i się samo robić, ale gupie nie chce

File: lab2/urdf/bogson.urdf.xacro (robot description, xacro)
@@ -5,79 +5,59 @@
   <xacro:property name="parameters" value="${load_yaml(find lab2)/parameters.yaml)}" />
   <xacro:property name="a1" value="${parameters['a1']}" />
-  <xacro:property name="a2" value="${parameters['a1']}" />
-  <xacro:property name="a3" value="${parameters['a1']}" />
+  <xacro:property name="a2" value="${parameters['a2']}" />
+  <xacro:property name="a3" value="${parameters['a3']}" />
   <!-- BGN - Robot description -->
   <xacro:link name="base"
-    originrpy="0 0 0"
     originxyz="0 0 0"
-    size="1 1 0.1"
-    material="magenta"
-    color="1 0 1 0.5">
+    dimensions="5 5 1">
+  </xacro:link>
+  <xacro:link name="link1"
+    originxyz="0 0 ${a1/2}"
+    dimensions="1 1 ${a1}">
   </xacro:link>
   <xacro:joint name="base_to_link1"
     type="revolute"
-    axis_xyz="0 0 1"
+    axis="0 0 1"
     originrpy="0 0 0"
-    originxyz="0 0 0.05"
+    originxyz="0 0 1"
     parent="base"
-    child="link1"
-    limitlow="-1.57" limithigh="1.57">
+    child="link1">
   </xacro:joint>
-  <xacro:link name="link1"
-    originxyz="${a1/2} 0 0"
+  <xacro:link name="link2"
+    originxyz="0 0 ${a2/2}"
+    dimensions="1 1 ${a2}">
+  </xacro:link>
+  <xacro:joint name="link1_to_link2"
+    type="revolute"
+    axis="0 0 1"
+    originrpy="0 0 ${1.57075}"
+    originxyz="0 0 ${a1}"
+    parent="link1"
+    child="link2">
+  </xacro:joint>
+  <xacro:link name="link3"
+    originxyz="0 0 ${a3/2}"
+    dimensions="1 1 ${a3}">
+  </xacro:link>
+  <xacro:joint name="link2_to_link3"
+    type="revolute"
+    axis="0 0 1"
     originrpy="0 0 0"
-    radius="0.05"
-    length="${a1}"
-    material="magenta"
-    color="1 0 1 0.5">
-  </xacro:link>
-  <xacro:joint name="link1-arm"
-    type="revolute"
-    axis_xyz="0 0 1"
-    originrpy="${-pi/2} 0 0"
-    originxyz="0 0 0"
-    parent="link1"
-    child="arm"
-    limitlow="-1.57" limithigh="1.57">
+    originxyz="0 0 ${a2}"
+    parent="link2"
+    child="link3">
   </xacro:joint>
-  <xacro:link name="arm"
-    originxyz="${pos2/2} 0 0"
-    originrpy="0 ${pi/2} 0"
-    radius="0.05"
-    length="${pos2}"
-    material="magenta"
-    color="1 0 1 0.5">
-  </xacro:link>
-  <xacro:joint name="arm-hand"
-    type="revolute"
-    axis_xyz="0 0 1"
-    originrpy="${-pi/2} 0 0"
-    originxyz="${a2} 0 0"
-    parent="arm"
-    child="hand"
-    limitlow="-2.90" limithigh="2.90">
-  </xacro:joint>
-  <xacro:link name="hand"
-    originxyz="${a3/2} 0 ${d3/2}"
-    originrpy="0 ${pi/2} 0"
-    radius="0.05"
-    length="${a3}"
-    material="magenta"
-    color="1 0 1 0.5">
+  <xacro:link name="narzedzie"
+    originxyz="0 0 0.5"
+    dimensions = "1 1 1">
   </xacro:link>
   <xacro:joint name="link3_to_narzedzie"
     type="revolute"
-    axis_xyz="0 0 1"
+    axis="0 0 1"
     originrpy="0 0 0"
-    originxyz="${a3} 0 0"
-    parent="hand"
-    child="tool"
-    limitlow="0" limithigh="0">
+    originxyz="0 0 ${a3}"
+    parent="link3"
+    child="narzedzie">
   </xacro:joint>
-  <xacro:link name="narzedzie"
-    originxyz="0 0 0"
-    originrpy="0 0 0"
-    size = 0.5 0.5 2">
-  </xacro:link>
   <!-- END - Robot description -->
 </robot>

File: lab2/urdf/bogson_template.urdf.xacro (robot description, xacro)
@@ -2,5 +2,5 @@
     <xacro:property name="DH" value="${load_yaml('DH.yaml')}"/>
     <xacro:property name="params" value="${load_yaml('rpy.yaml')}"/>
-    <xacro:macro name="link" params="name originxyz originrpy dimensions">
+    <xacro:macro name="link" params="name originxyz dimensions">
         <link name="${name}">
             <visual>
@@ -8,5 +8,5 @@
                     <box size="${dimensions}"/>
                 </geometry>
-                <origin rpy="${originrpy}" xyz="${originxyz}"/>
+                <origin rpy="0 0 0" xyz="${originxyz}"/>
                 <material name="magenta">
                     <color rgba="1 0 1 0.5"/>
@@ -16,7 +16,7 @@
     </xacro:macro>
     <xacro:macro name="joint" params=" name type axis parent child originxyz originrpy">
-        <joint name="base_to_link1" type="revolute">
+        <joint name="${name}" type="${type}">
             <axis xyz="${axis}"/>
-            <limit upper="5" lower="-5" effort="10" velocity="2" />
+            <limit upper="3.1415" lower="-3.1415" effort="10" velocity="2" />
             <parent link="${parent}"/>
             <child link="${child}"/>

Commit message: Próba zrobienia, żeby xacro działało
DISCLAIMER: NIE UDAŁO SIĘ, xacro wyrzuca 'invalid syntax', bo niby coś jest z parametrami, chyba, że nie może ich przeczytać, a raczej, że nie może ich potem użyć

File: lab2/urdf/bogson.urdf.xacro (robot description, xacro)
@@ -1,5 +1,5 @@
 <robot name="bogson" xmlns:xacro="http://www.ros.org/wiki/xacro">
   <!-- BGN - Include -->
-  <xacro:include filename="$(find lab2)/bogson_template.urdf.xacro" />
+  <xacro:include filename="$(find lab2)/bogson_template.urdf.xacro"/>
   <!-- END - Include -->
   <xacro:property name="parameters" value="${load_yaml(find lab2)/parameters.yaml)}" />
@@ -8,13 +8,13 @@
   <xacro:property name="a3" value="${parameters['a3']}" />
   <!-- BGN - Robot description -->
-  <xacro:link name="base"
+  <xacro:_link name="base"
     originxyz="0 0 0"
     dimensions="5 5 1">
-  </xacro:link>
-  <xacro:link name="link1"
+  </xacro:_link>
+  <xacro:_link name="link1"
     originxyz="0 0 ${a1/2}"
     dimensions="1 1 ${a1}">
-  </xacro:link>
-  <xacro:joint name="base_to_link1"
+  </xacro:_link>
+  <xacro:_joint name="base_to_link1"
     type="revolute"
     axis="0 0 1"
@@ -23,10 +23,10 @@
     parent="base"
     child="link1">
-  </xacro:joint>
-  <xacro:link name="link2"
+  </xacro:_joint>
+  <xacro:_link name="link2"
     originxyz="0 0 ${a2/2}"
     dimensions="1 1 ${a2}">
-  </xacro:link>
-  <xacro:joint name="link1_to_link2"
+  </xacro:_link>
+  <xacro:_joint name="link1_to_link2"
     type="revolute"
     axis="0 0 1"
@@ -35,10 +35,10 @@
     parent="link1"
     child="link2">
-  </xacro:joint>
-  <xacro:link name="link3"
+  </xacro:_joint>
+  <xacro:_link name="link3"
     originxyz="0 0 ${a3/2}"
     dimensions="1 1 ${a3}">
-  </xacro:link>
-  <xacro:joint name="link2_to_link3"
+  </xacro:_link>
+  <xacro:_joint name="link2_to_link3"
     type="revolute"
     axis="0 0 1"
@@ -47,10 +47,10 @@
     parent="link2"
     child="link3">
-  </xacro:joint>
-  <xacro:link name="narzedzie"
+  </xacro:_joint>
+  <xacro:_link name="narzedzie"
     originxyz="0 0 0.5"
-    dimensions = "1 1 1">
-  </xacro:link>
-  <xacro:joint name="link3_to_narzedzie"
+    dimensions="1 1 1">
+  </xacro:_link>
+  <xacro:_joint name="link3_to_narzedzie"
     type="revolute"
     axis="0 0 1"
@@ -59,5 +59,5 @@
     parent="link3"
     child="narzedzie">
-  </xacro:joint>
+  </xacro:_joint>
   <!-- END - Robot description -->
 </robot>

File: lab2/urdf/bogson_template.urdf.xacro (robot description, xacro)
@@ -1,6 +1,6 @@
 <robot name="bogson" xmlns:xacro="http://www.ros.org/wiki/xacro">
-    <xacro:property name="DH" value="${load_yaml('DH.yaml')}"/>
-    <xacro:property name="params" value="${load_yaml('rpy.yaml')}"/>
-    <xacro:macro name="link" params="name originxyz dimensions">
+    <!-- <xacro:property name="DH" value="${load_yaml('DH.yaml')}"/>
+    <xacro:property name="params" value="${load_yaml('rpy.yaml')}"/> -->
+    <xacro:macro name="_link" params="name dimensions originxyz">
         <link name="${name}">
             <visual>
@@ -15,8 +15,8 @@
         </link>
     </xacro:macro>
-    <xacro:macro name="joint" params=" name type axis parent child originxyz originrpy">
+    <xacro:macro name="_joint" params=" name type axis parent child originxyz originrpy">
         <joint name="${name}" type="${type}">
             <axis xyz="${axis}"/>
-            <limit upper="3.1415" lower="-3.1415" effort="10" velocity="2" />
+            <limit upper="3.1415" lower="-3.1415" effort="10" velocity="2"/>
             <parent link="${parent}"/>
             <child link="${child}"/>

Commit message: stylistyczne pierdoły

File: lab2/urdf/bogson.urdf.xacro (robot description, xacro)
@@ -3,8 +3,8 @@
   <xacro:include filename="$(find lab2)/bogson_template.urdf.xacro"/>
   <!-- END - Include -->
-  <xacro:property name="parameters" value="${load_yaml(find lab2)/parameters.yaml)}" />
-  <xacro:property name="a1" value="${parameters['a1']}" />
-  <xacro:property name="a2" value="${parameters['a2']}" />
-  <xacro:property name="a3" value="${parameters['a3']}" />
+  <xacro:property name="parameters" value="${load_yaml((find lab2)/parameters.yaml)}"/>
+  <xacro:property name="a1" value="${parameters['a1']}"/>
+  <xacro:property name="a2" value="${parameters['a2']}"/>
+  <xacro:property name="a3" value="${parameters['a3']}"/>
   <!-- BGN - Robot description -->
   <xacro:_link name="base"

Commit message: Revert "już powinno xacro działąć i się samo robić, ale gupie nie chce"
This reverts commit 15244f6bd0df4875602caf53aca67c09b48b793a.

File: lab2/urdf/bogson.urdf.xacro (robot description, xacro)
@@ -5,59 +5,79 @@
   <xacro:property name="parameters" value="${load_yaml(find lab2)/parameters.yaml)}" />
   <xacro:property name="a1" value="${parameters['a1']}" />
-  <xacro:property name="a2" value="${parameters['a2']}" />
-  <xacro:property name="a3" value="${parameters['a3']}" />
+  <xacro:property name="a2" value="${parameters['a1']}" />
+  <xacro:property name="a3" value="${parameters['a1']}" />
   <!-- BGN - Robot description -->
   <xacro:link name="base"
+    originrpy="0 0 0"
     originxyz="0 0 0"
-    dimensions="5 5 1">
-  </xacro:link>
-  <xacro:link name="link1"
-    originxyz="0 0 ${a1/2}"
-    dimensions="1 1 ${a1}">
+    size="1 1 0.1"
+    material="magenta"
+    color="1 0 1 0.5">
   </xacro:link>
   <xacro:joint name="base_to_link1"
     type="revolute"
-    axis="0 0 1"
+    axis_xyz="0 0 1"
     originrpy="0 0 0"
-    originxyz="0 0 1"
+    originxyz="0 0 0.05"
     parent="base"
-    child="link1">
+    child="link1"
+    limitlow="-1.57" limithigh="1.57">
   </xacro:joint>
-  <xacro:link name="link2"
-    originxyz="0 0 ${a2/2}"
-    dimensions="1 1 ${a2}">
+  <xacro:link name="link1"
+    originxyz="${a1/2} 0 0"
+    originrpy="0 0 0"
+    radius="0.05"
+    length="${a1}"
+    material="magenta"
+    color="1 0 1 0.5">
   </xacro:link>
-  <xacro:joint name="link1_to_link2"
+  <xacro:joint name="link1-arm"
     type="revolute"
-    axis="0 0 1"
-    originrpy="0 0 ${1.57075}"
-    originxyz="0 0 ${a1}"
+    axis_xyz="0 0 1"
+    originrpy="${-pi/2} 0 0"
+    originxyz="0 0 0"
     parent="link1"
-    child="link2">
+    child="arm"
+    limitlow="-1.57" limithigh="1.57">
   </xacro:joint>
-  <xacro:link name="link3"
-    originxyz="0 0 ${a3/2}"
-    dimensions="1 1 ${a3}">
+  <xacro:link name="arm"
+    originxyz="${pos2/2} 0 0"
+    originrpy="0 ${pi/2} 0"
+    radius="0.05"
+    length="${pos2}"
+    material="magenta"
+    color="1 0 1 0.5">
   </xacro:link>
-  <xacro:joint name="link2_to_link3"
+  <xacro:joint name="arm-hand"
     type="revolute"
-    axis="0 0 1"
-    originrpy="0 0 0"
-    originxyz="0 0 ${a2}"
-    parent="link2"
-    child="link3">
+    axis_xyz="0 0 1"
+    originrpy="${-pi/2} 0 0"
+    originxyz="${a2} 0 0"
+    parent="arm"
+    child="hand"
+    limitlow="-2.90" limithigh="2.90">
   </xacro:joint>
-  <xacro:link name="narzedzie"
-    originxyz="0 0 0.5"
-    dimensions = "1 1 1">
+  <xacro:link name="hand"
+    originxyz="${a3/2} 0 ${d3/2}"
+    originrpy="0 ${pi/2} 0"
+    radius="0.05"
+    length="${a3}"
+    material="magenta"
+    color="1 0 1 0.5">
   </xacro:link>
   <xacro:joint name="link3_to_narzedzie"
     type="revolute"
-    axis="0 0 1"
+    axis_xyz="0 0 1"
     originrpy="0 0 0"
-    originxyz="0 0 ${a3}"
-    parent="link3"
-    child="narzedzie">
+    originxyz="${a3} 0 0"
+    parent="hand"
+    child="tool"
+    limitlow="0" limithigh="0">
   </xacro:joint>
+  <xacro:link name="narzedzie"
+    originxyz="0 0 0"
+    originrpy="0 0 0"
+    size = 0.5 0.5 2">
+  </xacro:link>
   <!-- END - Robot description -->
 </robot>

File: lab2/urdf/bogson_template.urdf.xacro (robot description, xacro)
@@ -2,5 +2,5 @@
     <xacro:property name="DH" value="${load_yaml('DH.yaml')}"/>
     <xacro:property name="params" value="${load_yaml('rpy.yaml')}"/>
-    <xacro:macro name="link" params="name originxyz dimensions">
+    <xacro:macro name="link" params="name originxyz originrpy dimensions">
         <link name="${name}">
             <visual>
@@ -8,5 +8,5 @@
                     <box size="${dimensions}"/>
                 </geometry>
-                <origin rpy="0 0 0" xyz="${originxyz}"/>
+                <origin rpy="${originrpy}" xyz="${originxyz}"/>
                 <material name="magenta">
                     <color rgba="1 0 1 0.5"/>
@@ -16,7 +16,7 @@
     </xacro:macro>
     <xacro:macro name="joint" params=" name type axis parent child originxyz originrpy">
-        <joint name="${name}" type="${type}">
+        <joint name="base_to_link1" type="revolute">
             <axis xyz="${axis}"/>
-            <limit upper="3.1415" lower="-3.1415" effort="10" velocity="2" />
+            <limit upper="5" lower="-5" effort="10" velocity="2" />
             <parent link="${parent}"/>
             <child link="${child}"/>
